File: Projetos(Hardware)/LCD_TFT-Xplained_V1/LCD_TFT-Xplained_V1/LCD_TFT-Xplained_V1.sch (EAGLE design)
At the start: 11 parts

Commit message: Atualizacao LCD tft
Connections:
- removed net N$6: J3.8
- new net CS_OFF: J1.3
- new net GND_OFF: J1.1
- new net RST_OFF: J1.7
- new net VIN_OFF: J1.2
- new net X+_OFF: J1.9
- new net X-/SCL_OFF: J1.11
- new net Y+_OFF: J1.10
- new net Y-/SDA_OFF: J1.12
- net CS: no longer J1.3
- net GND: no longer J1.1
- net LITE: now also J3.8
- net RST: no longer J1.7
- net VIN: no longer J1.2
- net X+: no longer J1.9
- net X-/SCL: no longer J1.11
- net Y+: no longer J1.10
- net Y-/SDA: no longer J1.12
